Commit message: add

File: noor_robot/urdf/noor_robot.xacro (robot description, xacro)
@@ -1,8 +1,8 @@
 <?xml version='1.0'?>
 <robot name="noor_robot" xmlns:xacro="http://www.ros.org/wiki/xacro">
-  <link name="robot_footprint">
-  </link>
-  <joint name="robot_footprint_joint" type="fixed">
-      <parent link="robot_footprint"/>
+  <link name="base_footprint">
+  </link>
+  <joint name="base_footprint_joint" type="fixed">
+      <parent link="base_footprint"/>
       <child link="base_link"/>
   </joint>
